File: JTAG-Programmer.kicad_pcb (KiCad board)
At the start: 2 copper layers, 54.8 x 40.5 mm, 35 parts, among them J1 UJ2-MBH-1-SMT-TR, J2 Conn_02x05_Odd_Even, J3 Conn_02x05_Odd_Even, U1 FT2232HL, U2 93LC56C-I/SN, U4 TLV1117LV33DCYR, Y1 ASE-12.000MHZ-LC-T

Commit message: Small changes & added a readme
Routing:
- net +5V_USB: track 82.2 -> 80.6 mm
- net GND: track 35.9 -> 37.0 mm
